Commit message: 1

File: ridgeback/accessories.urdf.xacro (robot description, xacro)
@@ -9,7 +9,7 @@
     ridgeback_base/launch/base.launch
   -->
-  <xacro:include filename="$(find ridgeback_description)/urdf/accessories/sick_lms1xx_mount.urdf.xacro" />
-  <xacro:include filename="$(find ridgeback_description)/urdf/accessories/sick_s300_mount.urdf.xacro" />
-  <xacro:include filename="$(find ridgeback_description)/urdf/accessories/hokuyo_ust-10lx_mount.urdf.xacro" />
+  <xacro:include filename="$(find mobile_manipulator_description)/urdf/base/ridgeback/accessories/sick_lms1xx_mount.urdf.xacro" />
+  <xacro:include filename="$(find mobile_manipulator_description)/urdf/base/ridgeback/accessories/sick_s300_mount.urdf.xacro" />
+  <xacro:include filename="$(find mobile_manipulator_description)/urdf/base/ridgeback/accessories/hokuyo_ust-10lx_mount.urdf.xacro" />
   <!-- If enabled, generate the front HOKUYO UST-10LX LASER payload. -->
   <xacro:if value="$(optenv RIDGEBACK_FRONT_HOKUYO_LASER 0)">
@@ -51,5 +51,5 @@
   </xacro:if>
   <!-- Legacy support for Microstrain IMU GX2 -->
-  <xacro:include filename="$(find ridgeback_description)/urdf/accessories/microstrain_imu.urdf.xacro" />
+  <xacro:include filename="$(find mobile_manipulator_description)/urdf/base/ridgeback/accessories/microstrain_imu.urdf.xacro" />
   <xacro:if value="$(optenv RIDGEBACK_MICROSTRAIN_IMU 0)">
     <xacro:microstrain_imu prefix="$(optenv RIDGEBACK_MICROSTRAIN_IMU_PREFIX upgraded)"

File: ridgeback/accessories/hokuyo_ust-10lx_mount.urdf.xacro (robot description, xacro)
@@ -19,5 +19,5 @@
         <geometry>
           <!-- Origin of this mesh is the focal point of the LIDAR. -->
-          <mesh filename="package://ridgeback_description/meshes/ust-10lx.stl" />
+          <mesh filename="package://mobile_manipulation_description/meshes/base/ridgeback/ust-10lx.stl" />
         </geometry>
         <material name="dark_grey" />

File: ridgeback/accessories/microstrain_imu.urdf.xacro (robot description, xacro)
@@ -7,5 +7,5 @@
       <geometry>
         <!-- Origin of this mesh is the focal point of the LIDAR. -->
-        <mesh filename="package://ridgeback_description/meshes/3dm-gxX.stl" scale="0.001 0.001 0.001" />
+        <mesh filename="package://mobile_manipulation_description/meshes/base/ridgeback/3dm-gxX.stl" scale="0.001 0.001 0.001" />
       </geometry>
       <material name="dark_grey" />

File: ridgeback/ridgeback.urdf.xacro (robot description, xacro)
@@ -28,5 +28,5 @@
         <origin xyz="0 0 0" rpy="${PI/2} 0 0"/>
         <geometry>
-          <mesh filename="package://ridgeback_description/meshes/wheel.stl"/>
+          <mesh filename="package://mobile_manipulation_description/meshes/base/ridgeback/wheel.stl"/>
         </geometry>
         <material name="black" />
@@ -68,5 +68,5 @@
         <origin xyz="0 0 0" rpy="${PI/2} 0 ${PI/2}" />
         <geometry>
-          <mesh filename="package://ridgeback_description/meshes/rocker.stl"/>
+          <mesh filename="package://mobile_manipulation_description/meshes/base/ridgeback/rocker.stl"/>
         </geometry>
         <material name="black" />
@@ -111,5 +111,5 @@
       <origin xyz="0 0 0" rpy="0 0 0" />
       <geometry>
-        <mesh filename="package://ridgeback_description/meshes/body.stl"/>
+        <mesh filename="package://mobile_manipulation_description/meshes/base/ridgeback/body.stl"/>
       </geometry>
       <material name="black" />
@@ -118,5 +118,5 @@
       <origin xyz="0 0 0"/>
       <geometry>
-        <mesh filename="package://ridgeback_description/meshes/body-collision.stl"/>
+        <mesh filename="package://mobile_manipulation_description/meshes/base/ridgeback/body-collision.stl"/>
       </geometry>
     </collision>
@@ -164,5 +164,5 @@
       <origin xyz="0 0 0" rpy="0 0 ${PI}" />
       <geometry>
-        <mesh filename="package://ridgeback_description/meshes/side-cover.stl"/>
+        <mesh filename="package://mobile_manipulation_description/meshes/base/ridgeback/side-cover.stl"/>
       </geometry>
       <material name="yellow" />
@@ -173,5 +173,5 @@
       <origin xyz="0 0 0" rpy="0 0 0" />
       <geometry>
-        <mesh filename="package://ridgeback_description/meshes/side-cover.stl"/>
+        <mesh filename="package://mobile_manipulation_description/meshes/base/ridgeback/side-cover.stl"/>
       </geometry>
       <material name="yellow" />
@@ -187,5 +187,5 @@
       <origin xyz="0 0 0" rpy="0 0 0" />
       <geometry>
-        <mesh filename="package://ridgeback_description/meshes/end-cover.stl" />
+        <mesh filename="package://mobile_manipulation_description/meshes/base/ridgeback/end-cover.stl" />
       </geometry>
       <material name="black" />
@@ -201,5 +201,5 @@
       <origin xyz="0 0 0" rpy="0 0 ${PI}" />
       <geometry>
-        <mesh filename="package://ridgeback_description/meshes/end-cover.stl" />
+        <mesh filename="package://mobile_manipulation_description/meshes/base/ridgeback/end-cover.stl" />
       </geometry>
       <material name="black" />
@@ -220,5 +220,5 @@
       <origin xyz="0 0 0" rpy="0 0 0" />
       <geometry>
-        <mesh filename="package://ridgeback_description/meshes/lights.stl" />
+        <mesh filename="package://mobile_manipulation_description/meshes/base/ridgeback/lights.stl" />
       </geometry>
       <material name="white" />
@@ -229,5 +229,5 @@
       <origin xyz="0 0 0" rpy="0 0 ${PI}" />
       <geometry>
-        <mesh filename="package://ridgeback_description/meshes/lights.stl" />
+        <mesh filename="package://mobile_manipulation_description/meshes/base/ridgeback/lights.stl" />
       </geometry>
       <material name="black" />
@@ -243,5 +243,5 @@
       <origin xyz="0 0 0" rpy="0 0 0" />
       <geometry>
-        <mesh filename="package://ridgeback_description/meshes/top.stl" />
+        <mesh filename="package://mobile_manipulation_description/meshes/base/ridgeback/top.stl" />
       </geometry>
       <material name="black" />
@@ -250,5 +250,5 @@
       <origin xyz="0 0 0" rpy="0 0 0" />
       <geometry>
-        <mesh filename="package://ridgeback_description/meshes/top.stl"/>
+        <mesh filename="package://mobile_manipulation_description/meshes/base/ridgeback/top.stl"/>
       </geometry>
     </collision>
@@ -263,5 +263,5 @@
       <origin xyz="0 0 0" rpy="0 ${PI/2} 0" />
       <geometry>
-        <mesh filename="package://ridgeback_description/meshes/axle.stl" />
+        <mesh filename="package://mobile_manipulation_description/meshes/base/ridgeback/axle.stl" />
       </geometry>
       <material name="black" />
@@ -287,9 +287,9 @@
   </joint>
   <!-- Bring in simulation data for Gazebo. -->
-  <xacro:include filename="$(find ridgeback_description)/urdf/ridgeback.gazebo" />
+  <xacro:include filename="$(find mobile_manipulator_description)/urdf/base/ridgeback/ridgeback.gazebo" />
   <!-- Optional standard accessories, including their simulation data. The rendering
        of these into the final description is controlled by optenv variables, which
        default each one to off.-->
-  <xacro:include filename="$(find ridgeback_description)/urdf/accessories.urdf.xacro" />
+  <xacro:include filename="$(find mobile_manipulator_description)/urdf/base/ridgeback/accessories.urdf.xacro" />
   <!-- Optional custom includes. -->
   <xacro:include filename="$(optenv RIDGEBACK_URDF_EXTRAS empty.urdf)" />
