Commit message: 1

File: ridgeback/accessories/hokuyo_ust-10lx_mount.urdf.xacro (robot description, xacro)
@@ -19,5 +19,5 @@
         <geometry>
           <!-- Origin of this mesh is the focal point of the LIDAR. -->
-          <mesh filename="package://mobile_manipulation_description/meshes/base/ridgeback/ust-10lx.stl" />
+          <mesh filename="package://mobile_manipulator_description/meshes/base/ridgeback/ust-10lx.stl" />
         </geometry>
         <material name="dark_grey" />

File: ridgeback/accessories/microstrain_imu.urdf.xacro (robot description, xacro)
@@ -7,5 +7,5 @@
       <geometry>
         <!-- Origin of this mesh is the focal point of the LIDAR. -->
-        <mesh filename="package://mobile_manipulation_description/meshes/base/ridgeback/3dm-gxX.stl" scale="0.001 0.001 0.001" />
+        <mesh filename="package://mobile_manipulator_description/meshes/base/ridgeback/3dm-gxX.stl" scale="0.001 0.001 0.001" />
       </geometry>
       <material name="dark_grey" />

File: ridgeback/ridgeback.urdf.xacro (robot description, xacro)
@@ -28,5 +28,5 @@
         <origin xyz="0 0 0" rpy="${PI/2} 0 0"/>
         <geometry>
-          <mesh filename="package://mobile_manipulation_description/meshes/base/ridgeback/wheel.stl"/>
+          <mesh filename="package://mobile_manipulator_description/meshes/base/ridgeback/wheel.stl"/>
         </geometry>
         <material name="black" />
@@ -68,5 +68,5 @@
         <origin xyz="0 0 0" rpy="${PI/2} 0 ${PI/2}" />
         <geometry>
-          <mesh filename="package://mobile_manipulation_description/meshes/base/ridgeback/rocker.stl"/>
+          <mesh filename="package://mobile_manipulator_description/meshes/base/ridgeback/rocker.stl"/>
         </geometry>
         <material name="black" />
@@ -111,5 +111,5 @@
       <origin xyz="0 0 0" rpy="0 0 0" />
       <geometry>
-        <mesh filename="package://mobile_manipulation_description/meshes/base/ridgeback/body.stl"/>
+        <mesh filename="package://mobile_manipulator_description/meshes/base/ridgeback/body.stl"/>
       </geometry>
       <material name="black" />
@@ -118,5 +118,5 @@
       <origin xyz="0 0 0"/>
       <geometry>
-        <mesh filename="package://mobile_manipulation_description/meshes/base/ridgeback/body-collision.stl"/>
+        <mesh filename="package://mobile_manipulator_description/meshes/base/ridgeback/body-collision.stl"/>
       </geometry>
     </collision>
@@ -164,5 +164,5 @@
       <origin xyz="0 0 0" rpy="0 0 ${PI}" />
       <geometry>
-        <mesh filename="package://mobile_manipulation_description/meshes/base/ridgeback/side-cover.stl"/>
+        <mesh filename="package://mobile_manipulator_description/meshes/base/ridgeback/side-cover.stl"/>
       </geometry>
       <material name="yellow" />
@@ -173,5 +173,5 @@
       <origin xyz="0 0 0" rpy="0 0 0" />
       <geometry>
-        <mesh filename="package://mobile_manipulation_description/meshes/base/ridgeback/side-cover.stl"/>
+        <mesh filename="package://mobile_manipulator_description/meshes/base/ridgeback/side-cover.stl"/>
       </geometry>
       <material name="yellow" />
@@ -187,5 +187,5 @@
       <origin xyz="0 0 0" rpy="0 0 0" />
       <geometry>
-        <mesh filename="package://mobile_manipulation_description/meshes/base/ridgeback/end-cover.stl" />
+        <mesh filename="package://mobile_manipulator_description/meshes/base/ridgeback/end-cover.stl" />
       </geometry>
       <material name="black" />
@@ -201,5 +201,5 @@
       <origin xyz="0 0 0" rpy="0 0 ${PI}" />
       <geometry>
-        <mesh filename="package://mobile_manipulation_description/meshes/base/ridgeback/end-cover.stl" />
+        <mesh filename="package://mobile_manipulator_description/meshes/base/ridgeback/end-cover.stl" />
       </geometry>
       <material name="black" />
@@ -220,5 +220,5 @@
       <origin xyz="0 0 0" rpy="0 0 0" />
       <geometry>
-        <mesh filename="package://mobile_manipulation_description/meshes/base/ridgeback/lights.stl" />
+        <mesh filename="package://mobile_manipulator_description/meshes/base/ridgeback/lights.stl" />
       </geometry>
       <material name="white" />
@@ -229,5 +229,5 @@
       <origin xyz="0 0 0" rpy="0 0 ${PI}" />
       <geometry>
-        <mesh filename="package://mobile_manipulation_description/meshes/base/ridgeback/lights.stl" />
+        <mesh filename="package://mobile_manipulator_description/meshes/base/ridgeback/lights.stl" />
       </geometry>
       <material name="black" />
@@ -243,5 +243,5 @@
       <origin xyz="0 0 0" rpy="0 0 0" />
       <geometry>
-        <mesh filename="package://mobile_manipulation_description/meshes/base/ridgeback/top.stl" />
+        <mesh filename="package://mobile_manipulator_description/meshes/base/ridgeback/top.stl" />
       </geometry>
       <material name="black" />
@@ -250,5 +250,5 @@
       <origin xyz="0 0 0" rpy="0 0 0" />
       <geometry>
-        <mesh filename="package://mobile_manipulation_description/meshes/base/ridgeback/top.stl"/>
+        <mesh filename="package://mobile_manipulator_description/meshes/base/ridgeback/top.stl"/>
       </geometry>
     </collision>
@@ -263,5 +263,5 @@
       <origin xyz="0 0 0" rpy="0 ${PI/2} 0" />
       <geometry>
-        <mesh filename="package://mobile_manipulation_description/meshes/base/ridgeback/axle.stl" />
+        <mesh filename="package://mobile_manipulator_description/meshes/base/ridgeback/axle.stl" />
       </geometry>
       <material name="black" />
